File: PCB/node/Dendro.sch (EAGLE design)
At the start: 5 parts

Commit message: Summer 2022 Deployment Prep
Updated PCBs and code, includes Loom V3 and HypnosV3.3 changes
Parts:
- AS5311: value RJ45 -> JST-XH-05-PIN-ROUND-PAD; device SparkFun-Connectors:RJ45-8 -> Rembrandt Electronics - JST XH Connectors v1-0:JST-XH-05-PIN-ROUND-PAD
Connections:
- net A2 renamed LED
- removed net D11: BUTTON-1.S, MS1.GPIO11
- new net INT: BUTTON-1.S, MS1.GPIOA1
- net 3VRAIL: now also AS5311-1.S; no longer AS5311.1, AS5311.2
- net CSN: now also AS5311-4.S, MS1.GPIOA3; no longer AS5311.6, MS1.GPIO9
- net DO: now also AS5311-3.S; no longer AS5311.4
- net GND: now also AS5311-5.S; no longer AS5311.5
- net SCLK: now also AS5311-2.S; no longer AS5311.3
