File: PCB/node/Node_PCB_v20234.brd (EAGLE design)
At the start: 59.7 x 48.2 mm, 6 parts

Commit message: update PCB files
Parts:
- added TEROS: JST-XH-03-PIN-ROUND-PAD, Rembrandt Electronics - JST XH Connectors v1-0:JST-XH-03-PACKAGE-ROUND-PAD
- moved U$1 24.3 mm to (35.6, -3.81), turned to 0 degrees
- moved BUTTON 17.7 mm to (5.05, 17.1), turned to 270 degrees
- moved MS1 10.2 mm to (11.3, -2.74)
- moved NEOPIXEL 8.51 mm to (30.0, 36.9), turned to 180 degrees
- moved SHT30 6.58 mm to (47.0, 36.9), turned to 180 degrees
- moved AS5311 4.31 mm to (9.22, 30.6), turned to 270 degrees
Connections:
- new net A0: MS1.5, TEROS.3
- net 3VRAIL: now also TEROS.1
- net GND: now also TEROS.2
Routing:
- net A0: track 0.00 -> 24.9 mm
- net SDA: track 16.7 -> 26.0 mm, vias 0 -> 1
- net LED: track 51.4 -> 42.8 mm, vias 0 -> 1
- net SCL: track 15.2 -> 21.1 mm
- net SCLK: track 45.6 -> 51.1 mm
- net INT: track 28.7 -> 33.5 mm
- net DO: track 42.6 -> 46.7 mm, vias 1 -> 0
- net CSN: track 44.1 -> 42.9 mm, vias 1 -> 0
- added copper zone on layer 1, net 3VRAIL
- added copper zone on layer 16, net GND
- removed copper zone on layer 16, net 3VRAIL
- removed copper zone on layer 1, net GND
Other:
- board text added: "3V"
- board text added: "A0"
- board text added: "CLK"
- board text added: "CSN"
- board text added: "DATA"
- board text added: "DO"
- board text added: "Dendrometer V2023.4"
- board text added: "GND"
- board text added: "INT"
- board text added: "SCL"
- board text added: "SDA"
- board text removed: "< 3V"
- board text removed: "< CLK"
- board text removed: "< CSN"
- board text removed: "< DATA"
- board text removed: "< DO"
- board text removed: "< GND"
- board text removed: "< INT"
- board text removed: "< SCL"
- board text removed: "< SDA"
- board text removed: "Dendrometer V1.3"
