File: PCB/node/Node_PCB_v20234.sch (EAGLE design)
At the start: 5 parts

Commit message: update PCB files
Parts:
- added TEROS: JST-XH-03-PIN-ROUND-PAD, Rembrandt Electronics - JST XH Connectors v1-0:JST-XH-03-PIN-ROUND-PAD
Connections:
- new net A0: MS1.GPIOA0, TEROS-3.S
- net 3VRAIL: now also TEROS-1.S
- net GND: now also TEROS-2.S
